File: Hardware/cryptoshield.brd (EAGLE design)
At the start: 59.7 x 53.3 mm, 45 parts, among them J1 AVR_SPI_PRG_6PTH, Q1 BSS138, Q2 BSS138, U1 33mhz

Commit message: more work done, still work in progress
Parts:
- removed SJ3: JUMPER-PAD-2-NOYES_SILK, SparkFun-Passives:PAD-JUMPER-2-NO_YES_SILK
- added SJ1: (no value), SparkFun-Passives:PAD-JUMPER-2-NO_YES_SILK
- SJ2: value JUMPER-PAD-2-NOYES_SILK -> (none)
- moved SJ2 24.6 mm to (24.8, 5.08), flipped to the bottom, turned to 0 degrees
- moved S1 8.57 mm to (41.8, 29.0), turned to 180 degrees
- moved C3 6.73 mm to (39.1, 38.4)
- moved C4 5.84 mm to (57.9, 17.8)
- moved C6 5.84 mm to (57.9, 26.7)
- moved C9 5.84 mm to (57.9, 35.6)
- moved JP2 5.08 mm to (34.3, 39.4), turned to 270 degrees
- moved AES1 1.78 mm to (54.1, 17.8)
- moved ECC1 1.78 mm to (54.1, 35.6)
- moved SHA1 1.78 mm to (54.1, 26.7)
- moved RTC1 1.48 mm to (41.7, 34.8), turned to 270 degrees
- moved C12 0.13 mm to (44.7, 13.1)
- moved R6 0.13 mm to (44.7, 11.4)
Connections:
- removed net LV1: Q1.2, R3.2, SJ2.2
- removed net LV2: Q2.2, R1.2, SJ3.2
- new net N$4: SJ1.2, U$1.A4
- new net N$6: SJ2.2, U$1.A5
- net SCL: now also Q2.2, R1.2; no longer SJ3.1
- net SCL_IN: now also SJ2.1
- net SDA: now also Q1.2, R3.2; no longer SJ2.1
- net SDA_IN: now also SJ1.1
Routing:
- net 3.3V: track 12.9 -> 191.6 mm, vias 0 -> 8
- net SCL: track 0.00 -> 93.8 mm, vias 0 -> 3
- net SDA: track 0.00 -> 87.6 mm, vias 0 -> 3
- net N$6: track 0.00 -> 58.5 mm
- net N$4: track 0.00 -> 57.0 mm
- net SCL_IN: track 10.9 -> 39.4 mm
- net SDA_IN: track 8.22 -> 32.0 mm
- net ANT2: track 0.00 -> 17.1 mm
- net N$1: track 0.00 -> 15.4 mm
- net VBAT: track 0.00 -> 14.1 mm
- net PP: track 0.00 -> 13.0 mm
- net ANT1: track 0.00 -> 9.98 mm
- net 5V: track 0.00 -> 7.95 mm, vias 0 -> 2
- net SQW: track 0.00 -> 5.85 mm
- net 32KHZ: track 0.00 -> 5.85 mm
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Other:
- board text added: "I2C A4 A5"

Commit message: finished layout, ready for review
Connections:
- net 3.3V: no longer C1.1, C10.1, U$8.11, U$8.2
- net 5V: now also C1.1, C10.1, U$8.11, U$8.2
Routing:
- net 5V: track 7.95 -> 109.2 mm, vias 2 -> 5
- net 3.3V: track 191.6 -> 151.9 mm, vias 8 -> 6
- net GND: vias 3 -> 5
- added copper zone on layer 1, net 5V
Changed lines of the file:
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@@
 <setting verticaltext="up"/>
 </settings>
-<grid distance="0.005" unitdist="inch" unit="inch" style="lines" multiple="1" display="yes" altdistance="0.01" altunitdist="inch" altunit="inch"/>
+<grid distance="0.01" unitdist="inch" unit="inch" style="lines" multiple="1" display="yes" altdistance="0.01" altunitdist="inch" altunit="inch"/>
 <layers>
 <layer number="1" name="Top" color="4" fill="1" visible="yes" active="yes"/>
@@
 <text x="0.762" y="32.004" size="1.27" layer="22" font="vector" ratio="15" rot="SMR90">CryptoShield</text>
 <text x="2.54" y="18.034" size="1.27" layer="16" font="vector" ratio="15" rot="MR270" align="bottom-center">v01</text>
-<text x="50.8" y="-9.652" size="1.778" layer="51" ratio="15" rot="R180" align="bottom-right">Josh Datko / Casey Kuhns</text>
+<text x="54.61" y="-9.652" size="1.778" layer="51" ratio="15" rot="R180" align="bottom-right">Josh Datko / Casey Kuhns</text>
 <wire x1="57.15" y1="0" x2="59.69" y2="2.54" width="0.2032" layer="20"/>
 <wire x1="59.69" y1="2.54" x2="59.69" y2="50.8" width="0.2032" layer="20"/>
@@
 <vertex x="0" y="0"/>
 </polygon>
-<via x="45.085" y="28.321" extent="1-16" drill="0.508"/>
-<via x="46.101" y="31.877" extent="1-16" drill="0.508"/>
+<via x="46.228" y="28.194" extent="1-16" drill="0.508"/>
+<via x="46.228" y="30.988" extent="1-16" drill="0.508"/>
+<via x="47.498" y="30.988" extent="1-16" drill="0.508"/>
+<via x="47.498" y="28.194" extent="1-16" drill="0.508"/>
 </signal>
 <signal name="RST">
@@
 <contactref element="R1" pad="1"/>
 <contactref element="Q2" pad="1"/>
-<contactref element="U$8" pad="2"/>
 <contactref element="TPM1" pad="16"/>
 <wire x1="45.554" y1="11.43" x2="45.554" y2="13.081" width="0.2032" layer="1"/>
@@
 <wire x1="42.1132" y1="21.082" x2="42.1132" y2="22.8228" width="0.2032" layer="1"/>
 <wire x1="42.1132" y1="22.8228" x2="42.037" y2="22.899" width="0.2032" layer="1"/>
-<contactref element="U$8" pad="11"/>
 <contactref element="JP4" pad="6"/>
-<contactref element="C1" pad="1"/>
-<contactref element="C10" pad="1"/>
 <wire x1="54.29" y1="8.62" x2="54.29" y2="10.06" width="0.254" layer="1"/>
 <wire x1="54.29" y1="10.06" x2="54.19" y2="10.16" width="0.254" layer="1"/>
 <wire x1="49.21" y1="8.62" x2="49.21" y2="10.06" width="0.254" layer="1"/>
 <wire x1="49.21" y1="10.06" x2="49.11" y2="10.16" width="0.254" layer="1"/>
-<polygon width="0.254" layer="1">
-<vertex x="13.335" y="13.716"/>
-<vertex x="14.732" y="13.716"/>
-<vertex x="14.732" y="8.89"/>
-<vertex x="16.637" y="8.89"/>
-<vertex x="16.637" y="5.715"/>
-<vertex x="14.859" y="5.715"/>
-<vertex x="14.859" y="6.985"/>
-<vertex x="13.335" y="6.985"/>
-</polygon>
 <via x="56.007" y="17.145" extent="1-16" drill="0.508"/>
 <wire x1="56.007" y1="15.1638" x2="56.007" y2="17.145" width="0.254" layer="1"/>
@@
 <via x="56.007" y="26.035" extent="1-16" drill="0.508"/>
 <wire x1="56.007" y1="24.0538" x2="56.007" y2="26.035" width="0.254" layer="1"/>
-<via x="13.97" y="9.652" extent="1-16" drill="0.508"/>
-<wire x1="13.97" y1="9.652" x2="8.89" y2="14.732" width="0.4064" layer="16"/>
-<wire x1="8.89" y1="14.732" x2="8.89" y2="26.924" width="0.4064" layer="16"/>
-<wire x1="8.89" y1="26.924" x2="8.89" y2="34.29" width="0.4064" layer="16"/>
-<wire x1="20.0416" y1="24.9396" x2="20.0416" y2="26.5674" width="0.4064" layer="1"/>
-<wire x1="20.0416" y1="26.5674" x2="19.685" y2="26.924" width="0.4064" layer="1"/>
-<via x="19.685" y="26.924" extent="1-16" drill="0.508"/>
-<wire x1="19.685" y1="26.924" x2="8.89" y2="26.924" width="0.4064" layer="16"/>
 <wire x1="8.89" y1="34.29" x2="7.112" y2="36.068" width="0.4064" layer="16"/>
 <wire x1="7.112" y1="36.068" x2="7.112" y2="45.339" width="0.4064" layer="16"/>
@@
 <via x="55.88" y="11.176" extent="1-16" drill="0.508"/>
 <wire x1="55.88" y1="11.176" x2="55.88" y2="9.74" width="0.254" layer="1"/>
-<wire x1="50.8" y1="11.176" x2="30.48" y2="50.8" width="0" layer="19" extent="16-16"/>
+<contactref element="U$8" pad="2"/>
+<contactref element="U$8" pad="11"/>
+<contactref element="C1" pad="1"/>
+<contactref element="C10" pad="1"/>
+<polygon width="0.254" layer="1">
+<vertex x="13.335" y="13.716"/>
+<vertex x="14.732" y="13.716"/>
+<vertex x="14.732" y="8.89"/>
+<vertex x="16.637" y="8.89"/>
+<vertex x="16.637" y="5.715"/>
+<vertex x="14.859" y="5.715"/>
+<vertex x="14.859" y="6.985"/>
+<vertex x="13.335" y="6.985"/>
+</polygon>
+<via x="13.97" y="9.906" extent="1-16" drill="0.508"/>
+<wire x1="50.8" y1="11.176" x2="44.704" y2="5.08" width="0.254" layer="16"/>
+<wire x1="44.704" y1="5.08" x2="29.464" y2="5.08" width="0.254" layer="16"/>
+<wire x1="29.464" y1="5.08" x2="25.908" y2="8.636" width="0.254" layer="16"/>
+<wire x1="25.908" y1="8.636" x2="15.24" y2="8.636" width="0.254" layer="16"/>
+<wire x1="15.24" y1="8.636" x2="13.97" y2="9.906" width="0.254" layer="16"/>
+<wire x1="20.0416" y1="24.9396" x2="19.0976" y2="24.9396" width="0.254" layer="1"/>
+<wire x1="19.0976" y1="24.9396" x2="18.796" y2="24.638" width="0.254" layer="1"/>
+<via x="18.796" y="24.638" extent="1-16" drill="0.508"/>
+<wire x1="18.796" y1="24.638" x2="13.97" y2="19.812" width="0.254" layer="16"/>
+<wire x1="13.97" y1="19.812" x2="13.97" y2="9.906" width="0.254" layer="16"/>
+<wire x1="30.48" y1="50.8" x2="36.83" y2="44.45" width="0.254" layer="1"/>
+<wire x1="36.83" y1="44.45" x2="36.83" y2="40.132" width="0.254" layer="1"/>
+<via x="36.83" y="40.132" extent="1-16" drill="0.508"/>
+<wire x1="36.83" y1="40.132" x2="36.83" y2="33.274" width="0.254" layer="16"/>
+<wire x1="36.83" y1="33.274" x2="33.782" y2="30.226" width="0.254" layer="16"/>
+<wire x1="33.782" y1="30.226" x2="24.384" y2="30.226" width="0.254" layer="16"/>
+<wire x1="24.384" y1="30.226" x2="18.796" y2="24.638" width="0.254" layer="16"/>
 </signal>
 <signal name="SDA_IN">
